File: analog_input.kicad_sch (KiCad schematic)
At the start: 57 parts, among them J501 Conn_02x04_Odd_Even, J502 Conn_02x04, Q501 S9015, Q502 S9015, Q503 S9015, Q504 S9015, U501 LMV324, U502 ADS1115IDGS

Commit message: Fix DRC errors
Parts:
- FB501, FB502, FB503, FB504: symbol Device:Ferrite_Bead_Small -> Device:FerriteBead_Small
Changed lines of the file:
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@@
     (pin "2")
   )
-  (symbol (lib_id "Device:Ferrite_Bead_Small") (at 127 38.1 270) (unit 1)
+  (symbol (lib_id "Device:FerriteBead_Small") (at 127 38.1 270) (unit 1)
     (in_bom yes) (on_board yes)
     (property "Reference" "FB501" (id 0) (at 127 32.0802 90))
@@
     (pin "2")
   )
-  (symbol (lib_id "Device:Ferrite_Bead_Small") (at 127 60.96 270) (unit 1)
+  (symbol (lib_id "Device:FerriteBead_Small") (at 127 60.96 270) (unit 1)
     (in_bom yes) (on_board yes)
     (property "Reference" "FB502" (id 0) (at 127 54.9402 90))
@@
     (pin "2")
   )
-  (symbol (lib_id "Device:Ferrite_Bead_Small") (at 127 82.55 270) (unit 1)
+  (symbol (lib_id "Device:FerriteBead_Small") (at 127 82.55 270) (unit 1)
     (in_bom yes) (on_board yes)
     (property "Reference" "FB503" (id 0) (at 127 76.5302 90))
@@
     (pin "2")
   )
-  (symbol (lib_id "Device:Ferrite_Bead_Small") (at 127 105.41 270) (unit 1)
+  (symbol (lib_id "Device:FerriteBead_Small") (at 127 105.41 270) (unit 1)
     (in_bom yes) (on_board yes)
     (property "Reference" "FB504" (id 0) (at 127 99.3902 90))

Commit message: Add PCB graphics as symbols
Parts:
- JP202: renamed from JP502; footprint Jumper:SolderJumper-2_P1.3mm_Bridged_Pad1.0x1.5mm -> Jumper:SolderJumper-2_P1.3mm_Bridged2Bar_RoundedPad1.0x1.5mm
- renumbered C501 to C201, C502 to C202, C503 to C203, C504 to C204, C505 to C205, C506 to C206, C507 to C207, C508 to C208, C509 to C209, C510 to C210, C511 to C211, C512 to C212, C513 to C213, C514 to C214, C515 to C215, C516 to C216, C517 to C217, C518 to C218, C519 to C219, D501 to D201, D502 to D202, D503 to D203, D504 to D204, FB501 to FB201, FB502 to FB202, FB503 to FB203, FB504 to FB204, J501 to J201, J502 to J202, JP501 to JP201, JP503 to JP203, JP504 to JP204, Q501 to Q201, Q502 to Q202, Q503 to Q203, Q504 to Q204, R501 to R201, R502 to R202, R503 to R203, R504 to R204, R505 to R205, R506 to R206, R507 to R207, R508 to R208, R509 to R209, R510 to R210, R511 to R211, R512 to R212, R513 to R213, R514 to R214, R515 to R215, R516 to R216, R517 to R217, R518 to R218, U501 to U201, U502 to U202
Other:
- note added: "0x48"
- note added: "0x49"
- note added: "0x4a"
- note added: "0x4b"

Commit message: Replace C211-214 with 50V 0603 footprint parts
Parts:
- C207, C208, C209, C210: value 1uF -> 1uF/50V
- C211, C212, C213, C214: value 1uF -> 1uF/50V; footprint Capacitor_SMD:C_0402_1005Metric -> Capacitor_SMD:C_0603_1608Metric; LCSC C52923 -> C15849
Changed lines of the file:
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@@
     (pin "1")
   )
-  (symbol (lib_id "Device:C_Small") (at 121.92 41.91 0) (unit 1)
-    (in_bom yes) (on_board yes)
-    (property "Reference" "C207" (id 0) (at 124.2568 40.7416 0)
-      (effects (font (size 1.27 1.27)) (justify left))
-    )
-    (property "Value" "1uF" (id 1) (at 124.2568 43.053 0)
+  (symbol (lib_id "Device:C_Small") (at 121.92 41.91 0) (mirror y) (unit 1)
+    (in_bom yes) (on_board yes)
+    (property "Reference" "C207" (id 0) (at 119.5832 40.7416 0)
+      (effects (font (size 1.27 1.27)) (justify left))
+    )
+    (property "Value" "1uF/50V" (id 1) (at 119.5832 43.053 0)
       (effects (font (size 1.27 1.27)) (justify left))
     )
@@
       (effects (font (size 1.27 1.27)) (justify left))
     )
-    (property "Value" "1uF" (id 1) (at 134.4168 43.053 0)
-      (effects (font (size 1.27 1.27)) (justify left))
-    )
-    (property "Footprint" "Capacitor_SMD:C_0402_1005Metric" (id 2) (at 132.08 41.91 0)
+    (property "Value" "1uF/50V" (id 1) (at 134.4168 43.053 0)
+      (effects (font (size 1.27 1.27)) (justify left))
+    )
+    (property "Footprint" "Capacitor_SMD:C_0603_1608Metric" (id 2) (at 132.08 41.91 0)
       (effects (font (size 1.27 1.27)) hide)
     )
@@
       (effects (font (size 1.27 1.27)) hide)
     )
-    (property "LCSC" "C52923" (id 4) (at 132.08 41.91 0)
+    (property "LCSC" "C15849" (id 4) (at 132.08 41.91 0)
       (effects (font (size 1.27 1.27)) hide)
     )
@@
     (pin "1")
   )
-  (symbol (lib_id "Device:C_Small") (at 121.92 64.77 0) (unit 1)
-    (in_bom yes) (on_board yes)
-    (property "Reference" "C208" (id 0) (at 124.2568 63.6016 0)
-      (effects (font (size 1.27 1.27)) (justify left))
-    )
-    (property "Value" "1uF" (id 1) (at 124.2568 65.913 0)
+  (symbol (lib_id "Device:C_Small") (at 121.92 64.77 0) (mirror y) (unit 1)
+    (in_bom yes) (on_board yes)
+    (property "Reference" "C208" (id 0) (at 119.5832 63.6016 0)
+      (effects (font (size 1.27 1.27)) (justify left))
+    )
+    (property "Value" "1uF/50V" (id 1) (at 119.5832 65.913 0)
       (effects (font (size 1.27 1.27)) (justify left))
     )
@@
       (effects (font (size 1.27 1.27)) (justify left))
     )
-    (property "Value" "1uF" (id 1) (at 134.4168 65.913 0)
-      (effects (font (size 1.27 1.27)) (justify left))
-    )
-    (property "Footprint" "Capacitor_SMD:C_0402_1005Metric" (id 2) (at 132.08 64.77 0)
+    (property "Value" "1uF/50V" (id 1) (at 134.4168 65.913 0)
+      (effects (font (size 1.27 1.27)) (justify left))
+    )
+    (property "Footprint" "Capacitor_SMD:C_0603_1608Metric" (id 2) (at 132.08 64.77 0)
       (effects (font (size 1.27 1.27)) hide)
     )
@@
       (effects (font (size 1.27 1.27)) hide)
     )
-    (property "LCSC" "C52923" (id 4) (at 132.08 64.77 0)
+    (property "LCSC" "C15849" (id 4) (at 132.08 64.77 0)
       (effects (font (size 1.27 1.27)) hide)
     )
@@
     (pin "1")
   )
-  (symbol (lib_id "Device:C_Small") (at 121.92 86.36 0) (unit 1)
-    (in_bom yes) (on_board yes)
-    (property "Reference" "C209" (id 0) (at 124.2568 85.1916 0)
-      (effects (font (size 1.27 1.27)) (justify left))
-    )
-    (property "Value" "1uF" (id 1) (at 124.2568 87.503 0)
+  (symbol (lib_id "Device:C_Small") (at 121.92 86.36 0) (mirror y) (unit 1)
+    (in_bom yes) (on_board yes)
+    (property "Reference" "C209" (id 0) (at 119.5832 85.1916 0)
+      (effects (font (size 1.27 1.27)) (justify left))
+    )
+    (property "Value" "1uF/50V" (id 1) (at 119.5832 87.503 0)
       (effects (font (size 1.27 1.27)) (justify left))
     )
@@
       (effects (font (size 1.27 1.27)) (justify left))
     )
-    (property "Value" "1uF" (id 1) (at 134.4168 87.503 0)
-      (effects (font (size 1.27 1.27)) (justify left))
-    )
-    (property "Footprint" "Capacitor_SMD:C_0402_1005Metric" (id 2) (at 132.08 86.36 0)
+    (property "Value" "1uF/50V" (id 1) (at 134.4168 87.503 0)
+      (effects (font (size 1.27 1.27)) (justify left))
+    )
+    (property "Footprint" "Capacitor_SMD:C_0603_1608Metric" (id 2) (at 132.08 86.36 0)
       (effects (font (size 1.27 1.27)) hide)
     )
@@
       (effects (font (size 1.27 1.27)) hide)
     )
-    (property "LCSC" "C52923" (id 4) (at 132.08 86.36 0)
+    (property "LCSC" "C15849" (id 4) (at 132.08 86.36 0)
       (effects (font (size 1.27 1.27)) hide)
     )
@@
     (pin "1")
   )
-  (symbol (lib_id "Device:C_Small") (at 121.92 109.22 0) (unit 1)
-    (in_bom yes) (on_board yes)
-    (property "Reference" "C210" (id 0) (at 124.2568 108.0516 0)
-      (effects (font (size 1.27 1.27)) (justify left))
-    )
-    (property "Value" "1uF" (id 1) (at 124.2568 110.363 0)
+  (symbol (lib_id "Device:C_Small") (at 121.92 109.22 0) (mirror y) (unit 1)
+    (in_bom yes) (on_board yes)
+    (property "Reference" "C210" (id 0) (at 119.5832 108.0516 0)
+      (effects (font (size 1.27 1.27)) (justify left))
+    )
+    (property "Value" "1uF/50V" (id 1) (at 119.5832 110.363 0)
       (effects (font (size 1.27 1.27)) (justify left))
     )
@@
       (effects (font (size 1.27 1.27)) (justify left))
     )
-    (property "Value" "1uF" (id 1) (at 134.4168 110.363 0)
-      (effects (font (size 1.27 1.27)) (justify left))
-    )
-    (property "Footprint" "Capacitor_SMD:C_0402_1005Metric" (id 2) (at 132.08 109.22 0)
+    (property "Value" "1uF/50V" (id 1) (at 134.4168 110.363 0)
+      (effects (font (size 1.27 1.27)) (justify left))
+    )
+    (property "Footprint" "Capacitor_SMD:C_0603_1608Metric" (id 2) (at 132.08 109.22 0)
       (effects (font (size 1.27 1.27)) hide)
     )
@@
       (effects (font (size 1.27 1.27)) hide)
     )
-    (property "LCSC" "C52923" (id 4) (at 132.08 109.22 0)
-      (effects (font (size 1.27 1.27)) hide)
-    )
+    (property "LCSC" "C15849" (id 4) (at 132.08 109.22 0)
+      (effects (font (size 1.27 1.27)) hide)
+    )
