File: digital_input.kicad_sch (KiCad schematic)
At the start: 34 parts, among them J301 Conn_02x04_Odd_Even, J302 Conn_02x04_Odd_Even

Commit message: Fix DRC errors
Parts:
- FB301, FB302, FB303, FB304: symbol Device:Ferrite_Bead_Small -> Device:FerriteBead_Small
Changed lines of the file:
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@@
     (pin "1")
   )
-  (symbol (lib_id "Device:C_Small") (at 95.25 43.18 0) (mirror y)
+  (symbol (lib_id "Device:C_Small") (at 95.25 43.18 0) (mirror y) (unit 1)
     (in_bom yes) (on_board yes)
     (property "Reference" "C301" (id 0) (at 92.9132 42.0116 0)
@@
     (pin "2")
   )
-  (symbol (lib_id "Device:C_Small") (at 105.41 43.18 0)
+  (symbol (lib_id "Device:C_Small") (at 105.41 43.18 0) (unit 1)
     (in_bom yes) (on_board yes)
     (property "Reference" "C305" (id 0) (at 107.7468 42.0116 0)
@@
     (pin "2")
   )
-  (symbol (lib_id "Device:Ferrite_Bead_Small") (at 100.33 39.37 270)
+  (symbol (lib_id "Device:FerriteBead_Small") (at 100.33 39.37 270) (unit 1)
     (in_bom yes) (on_board yes)
     (property "Reference" "FB301" (id 0) (at 100.33 33.3502 90))
@@
     (pin "2")
   )
-  (symbol (lib_id "power:GND") (at 95.25 46.99 0)
+  (symbol (lib_id "power:GND") (at 95.25 46.99 0) (unit 1)
     (in_bom yes) (on_board yes)
     (property "Reference" "#PWR0302" (id 0) (at 95.25 53.34 0)
@@
     (pin "1")
   )
-  (symbol (lib_id "power:GND") (at 105.41 46.99 0)
+  (symbol (lib_id "power:GND") (at 105.41 46.99 0) (unit 1)
     (in_bom yes) (on_board yes)
     (property "Reference" "#PWR0306" (id 0) (at 105.41 53.34 0)
@@
     (pin "1")
   )
-  (symbol (lib_id "Device:C_Small") (at 95.25 77.47 0) (mirror y)
+  (symbol (lib_id "Device:C_Small") (at 95.25 77.47 0) (mirror y) (unit 1)
     (in_bom yes) (on_board yes)
     (property "Reference" "C302" (id 0) (at 92.9132 76.3016 0)
@@
     (pin "2")
   )
-  (symbol (lib_id "Device:C_Small") (at 105.41 77.47 0)
+  (symbol (lib_id "Device:C_Small") (at 105.41 77.47 0) (unit 1)
     (in_bom yes) (on_board yes)
     (property "Reference" "C306" (id 0) (at 107.7468 76.3016 0)
@@
     (pin "2")
   )
-  (symbol (lib_id "Device:Ferrite_Bead_Small") (at 100.33 73.66 270)
+  (symbol (lib_id "Device:FerriteBead_Small") (at 100.33 73.66 270) (unit 1)
     (in_bom yes) (on_board yes)
     (property "Reference" "FB302" (id 0) (at 100.33 67.6402 90))
@@
     (pin "2")
   )
-  (symbol (lib_id "power:GND") (at 95.25 81.28 0)
+  (symbol (lib_id "power:GND") (at 95.25 81.28 0) (unit 1)
     (in_bom yes) (on_board yes)
     (property "Reference" "#PWR0303" (id 0) (at 95.25 87.63 0)
@@
     (pin "1")
   )
-  (symbol (lib_id "power:GND") (at 105.41 81.28 0)
+  (symbol (lib_id "power:GND") (at 105.41 81.28 0) (unit 1)
     (in_bom yes) (on_board yes)
     (property "Reference" "#PWR0307" (id 0) (at 105.41 87.63 0)
@@
     (pin "1")
   )
-  (symbol (lib_id "Device:C_Small") (at 95.25 111.76 0) (mirror y)
+  (symbol (lib_id "Device:C_Small") (at 95.25 111.76 0) (mirror y) (unit 1)
     (in_bom yes) (on_board yes)
     (property "Reference" "C303" (id 0) (at 92.9132 110.5916 0)
@@
     (pin "2")
   )
-  (symbol (lib_id "Device:C_Small") (at 105.41 111.76 0)
+  (symbol (lib_id "Device:C_Small") (at 105.41 111.76 0) (unit 1)
     (in_bom yes) (on_board yes)
     (property "Reference" "C307" (id 0) (at 107.7468 110.5916 0)
@@
     (pin "2")
   )
-  (symbol (lib_id "Device:Ferrite_Bead_Small") (at 100.33 107.95 270)
+  (symbol (lib_id "Device:FerriteBead_Small") (at 100.33 107.95 270) (unit 1)
     (in_bom yes) (on_board yes)
     (property "Reference" "FB303" (id 0) (at 100.33 101.9302 90))
@@
     (pin "2")
   )
-  (symbol (lib_id "power:GND") (at 95.25 115.57 0)
+  (symbol (lib_id "power:GND") (at 95.25 115.57 0) (unit 1)
     (in_bom yes) (on_board yes)
     (property "Reference" "#PWR0304" (id 0) (at 95.25 121.92 0)
@@
     (pin "1")
   )
-  (symbol (lib_id "power:GND") (at 105.41 115.57 0)
+  (symbol (lib_id "power:GND") (at 105.41 115.57 0) (unit 1)
     (in_bom yes) (on_board yes)
     (property "Reference" "#PWR0308" (id 0) (at 105.41 121.92 0)
@@
     (pin "1")
   )
-  (symbol (lib_id "Device:C_Small") (at 95.25 146.05 0) (mirror y)
+  (symbol (lib_id "Device:C_Small") (at 95.25 146.05 0) (mirror y) (unit 1)
     (in_bom yes) (on_board yes)
     (property "Reference" "C304" (id 0) (at 92.9132 144.8816 0)
@@
     (pin "2")
   )
-  (symbol (lib_id "Device:C_Small") (at 105.41 146.05 0)
+  (symbol (lib_id "Device:C_Small") (at 105.41 146.05 0) (unit 1)
     (in_bom yes) (on_board yes)
     (property "Reference" "C308" (id 0) (at 107.7468 144.8816 0)
@@
     (pin "2")
   )
-  (symbol (lib_id "Device:Ferrite_Bead_Small") (at 100.33 142.24 270)
+  (symbol (lib_id "Device:FerriteBead_Small") (at 100.33 142.24 270) (unit 1)
     (in_bom yes) (on_board yes)
     (property "Reference" "FB304" (id 0) (at 100.33 136.2202 90))
@@
     (pin "2")
   )
-  (symbol (lib_id "power:GND") (at 95.25 149.86 0)
+  (symbol (lib_id "power:GND") (at 95.25 149.86 0) (unit 1)
     (in_bom yes) (on_board yes)
     (property "Reference" "#PWR0305" (id 0) (at 95.25 156.21 0)
@@
     (pin "1")
   )
-  (symbol (lib_id "power:GND") (at 105.41 149.86 0)
+  (symbol (lib_id "power:GND") (at 105.41 149.86 0) (unit 1)
     (in_bom yes) (on_board yes)
     (property "Reference" "#PWR0309" (id 0) (at 105.41 156.21 0)
